File: hardware/0.1/keyboard.kicad_sch (KiCad schematic)
At the start: 322 parts, among them J1 USB_C_Receptacle_USB2.0, J2 SWD, J3 SPARE, Q1 BSS138, Q2 DTC123J, SW1 RotaryEncoder_Switch, SW10 KEYSW, SW100 KEYSW, SW101 KEYSW, SW102 KEYSW, SW103 KEYSW, SW104 KEYSW, SW105 KEYSW, SW106 KEYSW, SW107 KEYSW, SW108 KEYSW, SW109 KEYSW, SW11 KEYSW, SW110 KEYSW, SW111 KEYSW, SW112 KEYSW, SW113 KEYSW, SW114 KEYSW, SW115 KEYSW, SW116 KEYSW, SW117 KEYSW, SW118 KEYSW, SW119 KEYSW, SW12 KEYSW, SW120 KEYSW, SW121 KEYSW, SW122 KEYSW, SW123 KEYSW, SW124 RotaryEncoder_Switch, SW125 KEYSW, SW126 KEYSW, SW127 KEYSW, SW128 KEYSW, SW129 KEYSW, SW13 KEYSW, SW14 KEYSW, SW15 KEYSW, SW16 KEYSW, SW17 KEYSW, SW18 KEYSW, SW19 KEYSW, SW2 KEYSW, SW20 KEYSW, SW21 KEYSW, SW22 KEYSW, SW23 KEYSW, SW24 KEYSW, SW25 KEYSW, SW26 KEYSW, SW27 KEYSW, SW28 KEYSW, SW29 KEYSW, SW3 KEYSW, SW30 KEYSW, SW31 KEYSW, SW32 KEYSW, SW33 KEYSW, SW34 KEYSW, SW35 KEYSW, SW36 KEYSW, SW37 KEYSW, SW38 KEYSW, SW39 KEYSW, SW4 KEYSW, SW40 KEYSW, SW41 KEYSW, SW42 KEYSW, SW43 KEYSW, SW44 KEYSW, SW45 KEYSW, SW46 KEYSW, SW47 KEYSW, SW48 KEYSW, SW49 KEYSW, SW5 KEYSW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

Commit message: 0.1 off to fab
Parts:
- added LOGO2: LOUISE, louise-footprints:louise, symbol Graphic:SYM_LASER_Small
- added R8: 22R, Resistor_SMD:R_0603_1608Metric, symbol Device:R
- BZ1: footprint Buzzer_Beeper:Buzzer_Murata_PKMCS0909E -> josh-mechanical:Buzzer_Murata_PKMCS0909E; MPN (none) -> PKMCS0909E; Manufacturer (none) -> Murata Electronics
- C1, C10, C11, C13, C14, C16, C17, C18, C19, C2, C20, C21, C22, C23, C3, C30, C31, C32, C33, C34, C35, C36, C4, C5, C6, C8, C9: LCSC (none) -> C14663; MPN (none) -> CC0603KRX7R9BB104; Manufacturer (none) -> YAGEO
- C12, C15, C24, C28, C29, C7: LCSC (none) -> C19666; MPN (none) -> CL10A475KO8NNNC; Manufacturer (none) -> Samsung Electro-Mechanics
- C25: LCSC (none) -> C96446; MPN (none) -> CL10A106MA8NRNC; Manufacturer (none) -> Samsung Electro-Mechanics
- C26, C27: LCSC (none) -> C1644; MPN (none) -> CL10C150JB8NNNC; Manufacturer (none) -> Samsung Electro-Mechanics
- D1, D100, D101, D102, D103, D104, D105, D106, D107, D108, D109, D11, D110, D111, D112, D113, D114, D115, D116, D117, D118, D119, D12, D120, D121, D122, D123, D124, D125, D126, D127, D128, D129, D13, D130, D131, D132, D133, D14, D15, D16, D2, D21, D22, D23, D24, D25, D26, D29, D3, D30, D31, D32, D33, D34, D38, D39, D4, D40, D41, D42, D43, D47, D48, D49, D5, D50, D54, D55, D56, D57, D58, D59, D6, D61, D62, D63, D64, D65, D66, D67, D68, D69, D70, D71, D72, D73, D74, D75, D76, D77, D78, D79, D80, D81, D82, D83, D84, D85, D86, D87, D88, D89, D90, D91, D92, D93, D94, D95, D96, D98, D99: LCSC (none) -> C81598; MPN (none) -> 1N4148W; Manufacturer (none) -> Semtech
- D10, D134, D135, D17, D18, D19, D20, D27, D28, D35, D36, D37, D45, D51, D53, D7, D8, D9: LCSC (none) -> C2761795; MPN (none) -> WS2812B-B/W; Manufacturer (none) -> Worldsemi
- D44, D46, D52, D60: MPN (none) -> SK6812-MINI-E; Manufacturer (none) -> Shenzhen LED Color
- D97: value LED_RED -> BLUE; LCSC (none) -> C72041; MPN (none) -> 19-217/BHC-ZL1M2RY/3T; Manufacturer (none) -> Everlight Elec
- F1: LCSC (none) -> C66452; MPN (none) -> SMD0805-050; Manufacturer (none) -> TECHFUSE
- H1, H2, J2, J3, JP1, LOGO3, SW1, SW10, SW100, SW101, SW102, SW103, SW104, SW105, SW106, SW107, SW108, SW109, SW11, SW110, SW111, SW112, SW113, SW114, SW115, SW116, SW117, SW118, SW119, SW12, SW120, SW121, SW122, SW123, SW124, SW125, SW126, SW127, SW128, SW129, SW13, SW14, SW15, SW16, SW17, SW18, SW19, SW2, SW20, SW21, SW22, SW23, SW24, SW25, SW26, SW27, SW28, SW29, SW3, SW30, SW31, SW32, SW33, SW34, SW35, SW36, SW37, SW38, SW39, SW4, SW40, SW41, SW42, SW43, SW44, SW45, SW46, SW47, SW48, SW49, SW5, SW50, SW51, SW52, SW53, SW54, SW55, SW56, SW58, SW59, SW6, SW60, SW61, SW62, SW63, SW64, SW65, SW66, SW67, SW68, SW69, SW7, SW70, SW71, SW72, SW73, SW74, SW75, SW76, SW77, SW78, SW79, SW8, SW80, SW81, SW82, SW83, SW84, SW85, SW86, SW87, SW88, SW89, SW9, SW90, SW91, SW92, SW93, SW94, SW95, SW96, SW97, SW98, SW99: DNP (none) -> DNP
- J1: LCSC (none) -> C165948; MPN (none) -> TYPE-C-31-M-12; Manufacturer (none) -> Korean Hroparts Elec
- Q1: value BSS138 -> 2N7002; LCSC (none) -> C8545; MPN (none) -> 2N7002; Manufacturer (none) -> Changjiang Electronics Tech (CJ)
- Q2: LCSC (none) -> C145108; MPN (none) -> DDTC123JCA-7-F; Manufacturer (none) -> Diodes Incorporated
- R1, R2, R3, R4, R6: LCSC (none) -> C23186; MPN (none) -> 0603WAF5101T5E; Manufacturer (none) -> UNI-ROYAL(Uniroyal Elec)
- R5: LCSC (none) -> C25803; MPN (none) -> 0603WAF1003T5E; Manufacturer (none) -> UNI-ROYAL(Uniroyal Elec)
- R7: LCSC (none) -> C22843; MPN (none) -> 0603WAF1501T5E; Manufacturer (none) -> UNI-ROYAL(Uniroyal Elec)
- SW57: LCSC (none) -> C99271; MPN (none) -> KMR231GLFS; Manufacturer (none) -> C&K
- U1: LCSC (none) -> C85364; MPN (none) -> XC6206P332MR; Manufacturer (none) -> ProTek Devices
- U2: LCSC (none) -> C5446; MPN (none) -> XC6206P332MR; Manufacturer (none) -> Torex Semicon
- U3: value STM32F303RCTx -> STM32F303CBT6; LCSC (none) -> C108516; MPN (none) -> STM32F303CBT6; Manufacturer (none) -> STMicroelectronics
- Y1: LCSC (none) -> C403948; MPN (none) -> TAXM8M4RFDCET2T; Manufacturer (none) -> TAE(Zhejiang Abel Elec)
Connections:
- net BUZZER: now also R8.1; no longer BZ1.1 (-)
- new net: BZ1.1 (-), R8.2
- no-connect marks 9 -> 16
Other:
- moved on the sheet: BZ1

Commit message: bom fix
Parts:
- H1, H2, J2, JP1: now left out of the parts list
- U3: value STM32F303CBT6 -> STM32F303RBT6; LCSC C108516 -> C130453; MPN STM32F303CBT6 -> STM32F303RBT6
Changed lines of the file:
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@@
     (in_bom yes) (on_board yes)
     (property "Reference" "U3" (id 0) (at 341.63 246.38 0))
-    (property "Value" "STM32F303CBT6" (id 1) (at 355.6 290.83 90))
+    (property "Value" "STM32F303RBT6" (id 1) (at 355.6 290.83 90))
     (property "Footprint" "Package_QFP:LQFP-64_10x10mm_P0.5mm" (id 2) (at 340.36 334.01 0)
       (effects (font (size 1.27 1.27)) (justify right) hide)
@@
       (effects (font (size 1.27 1.27)) hide)
     )
-    (property "LCSC" "C108516" (id 4) (at 355.6 290.83 0)
+    (property "LCSC" "C130453" (id 4) (at 355.6 290.83 0)
       (effects (font (size 1.27 1.27)) hide)
     )
-    (property "MPN" "STM32F303CBT6" (id 5) (at 355.6 290.83 0)
+    (property "MPN" "STM32F303RBT6" (id 5) (at 355.6 290.83 0)
       (effects (font (size 1.27 1.27)) hide)
     )
@@
   )
   (symbol (lib_id "Connector:Conn_01x05_Male") (at 342.9 401.32 0) (unit 1)
-    (in_bom yes) (on_board yes)
+    (in_bom no) (on_board yes)
     (property "Reference" "J2" (id 0) (at 343.535 391.16 0))
     (property "Value" "SWD" (id 1) (at 344.17 393.7 0))
@@
   )
   (symbol (lib_id "Mechanical:MountingHole_Pad") (at 378.46 397.51 90) (unit 1)
-    (in_bom yes) (on_board yes)
+    (in_bom no) (on_board yes)
     (property "Reference" "H2" (id 0) (at 372.11 396.24 90))
     (property "Value" "M2" (id 1) (at 372.11 398.78 90))
@@
   )
   (symbol (lib_id "Mechanical:MountingHole_Pad") (at 378.46 392.43 90) (unit 1)
-    (in_bom yes) (on_board yes)
+    (in_bom no) (on_board yes)
     (property "Reference" "H1" (id 0) (at 372.11 391.16 90))
     (property "Value" "M2" (id 1) (at 372.11 393.7 90))
@@
   )
   (symbol (lib_id "Jumper:Jumper_2_Bridged") (at 152.4 228.6 90) (unit 1)
-    (in_bom yes) (on_board yes) (fields_autoplaced)
+    (in_bom no) (on_board yes) (fields_autoplaced)
     (property "Reference" "JP1" (id 0) (at 153.67 227.3299 90)
       (effects (font (size 1.27 1.27)) (justify right))
@@
     )
     (path "/00000000-0000-0000-0000-000067341156"
-      (reference "U3") (unit 1) (value "STM32F303CBT6") (footprint "Package_QFP:LQFP-64_10x10mm_P0.5mm")
+      (reference "U3") (unit 1) (value "STM32F303RBT6") (footprint "Package_QFP:LQFP-64_10x10mm_P0.5mm")
     )
     (path "/00000000-0000-0000-0000-000069fe5765"
